File: Particle2NodeMCU.brd (EAGLE design)
At the start: 25.4 x 48.3 mm, 9 parts, among them Q1 MOSFET-N, Q2 MOSFET-N

Commit message: Updated to 1.1a
Parts:
- added JP4: (no value), SparkFun-Connectors:1X15
- JP2: device SparkFun-Connectors:1X15 -> SparkFun-Connectors:1X02_LOCK
- moved JP2 39.3 mm to (22.9, 46.9), turned to 180 degrees
- moved LOGO2 1.27 mm to (12.7, 12.7)
Connections:
- net GPIO2 renamed GPIO15
- net TINFO-ESP renamed TINFO-ADAPTER
- net 3V3: now also JP4.11; no longer JP2.11
- net A0: now also JP4.1; no longer JP2.1
- net GND: now also JP4.10, JP4.14; no longer JP2.10, JP2.14
- net GPIO3: now also JP2.2
- net RST: now also JP4.13; no longer JP2.13
- net TINFO: now also JP2.1
- net VIN: now also JP4.15; no longer JP2.15
Routing:
- net TINFO: track 18.7 -> 40.5 mm
- net GPIO3: track 13.0 -> 33.1 mm
- net GND: track 15.5 -> 0.00 mm
Other:
- board text added: "3V3"
- board text added: "For Téléinfo you need to : Close JP1 If Remora PCB is < v1.3 Close JP2 If Remora PCB is >= v1.3 Q2/Q3/R3 not needed in this case"
- board text added: "JP2"
- board text added: "Open JP1 & JP2 to upload"
- board text added: "Particle NodeMCU Adapter V1.1a"
- board text added: "Particle Spark/Photon NodeMCU Adapter V1.1a"
- board text added: "VIN"
- board text removed: "Node 3V3"
- board text removed: "Node VIN"
- board text removed: "Open to upload Close Téléinfo"
- board text removed: "Open to upload firmware Close to enable Téléinfo"
- board text removed: "Particle NodeMCU Adapter V1.1"
- board text removed: "Particle Spark/Photon NodeMCU Adapter V1.1"

Commit message: Ready To Panelize
Connections:
- net 3V3: no longer JP3.6
Routing:
- net 3V3: track 59.6 -> 33.2 mm, vias 2 -> 0
Other:
- board text added: "Q1"
- board text added: "Q2"
- board text added: "R1"
